File: kicad/expansion_board.kicad_pcb (KiCad board)
At the start: 2 copper layers, 14 parts, among them J1 Conn_01x08, J2 Conn_01x06, J3 Conn_01x02, J4 Conn_01x04_Female, J5 Conn_01x04_Female, J6 Conn_01x04_Female, J7 Conn_01x08, J8 Conn_01x10, SW1 SW_Push

Commit message: update
Parts:
- removed D2: LED blue, expansion_board:LED
- removed R2: 470, expansion_board:Register
- SW1: footprint expansion_board:Tactile switch 4P -> expansion_board:Tactile_switch_4P
- moved J3 12.7 mm to (139.6, 105.7)
- moved R1 10.9 mm to (182.8, 105.7), turned to 90 degrees
- moved D1 3.59 mm to (182.8, 93.0)
- moved C1 2.54 mm to (142.2, 95.5)
- moved J4 2.54 mm to (187.9, 93.0)
- moved J6 2.54 mm to (198.1, 93.0)
- moved SW1 1.80 mm to (148.5, 94.2)
Connections:
- SW1 pad 2: (no net) -> GND
- SW1 pad 3: GND -> (no net)
Routing:
- net Net-(J7-Pad5): track 83.8 -> 0.00 mm
- net Net-(J3-Pad1): track 68.6 -> 99.1 mm
- net Net-(J7-Pad6): track 78.7 -> 55.9 mm
- net Net-(D2-Pad1): track 15.2 -> 0.00 mm
- net GND: track 78.7 -> 91.4 mm, vias 2 -> 0
- net Net-(D1-Pad1): track 12.7 -> 7.62 mm
- net Net-(J6-Pad4): track 71.1 -> 68.6 mm
- net +3V3: track 50.8 -> 53.3 mm, vias 2 -> 0
- net Net-(C1-Pad2): track 38.1 -> 40.6 mm

Commit message: reciver
Parts:
- moved J6 2.54 mm to (195.5, 93.0)
Routing:
- net Net-(J6-Pad4): track 68.6 -> 66.0 mm
- net +3V3: track 53.3 -> 50.8 mm
Changed lines of the file:
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@@
     (links 16)
     (no_connects 1)
-    (area 0 0 0 0)
+    (area 136.1215 83.099 201.6715 138.489)
     (thickness 1.6)
     (drawings 0)
@@
   )
   (module "expansion_board:Pin Header 4P" (layer F.Cu)
-    (at 198.0565 92.964 270)
+    (at 195.5165 92.964 270)
     (fp_text reference J6 (at 0 2.54 270) (layer F.SilkS)
       (effects (font (size 1 1) (thickness 0.15)))
@@
   )
   (segment (start 154.8765 91.694) (end 154.8765 91.694) (width 0.25) (layer F.Cu) (net 0) (status 30))
-  (segment (start 144.7165 96.774) (end 144.7165 99.314) (width 0.25) (layer B.Cu) (net 1) (status 400000))
+  (segment (start 144.7165 96.774) (end 144.7165 99.314) (width 0.25) (layer B.Cu) (net 1))
   (segment (start 144.7165 104.394) (end 144.7165 99.314) (width 0.25) (layer B.Cu) (net 1))
   (segment (start 144.7165 104.394) (end 159.9565 104.394) (width 0.25) (layer B.Cu) (net 1))
@@
   (segment (start 175.1965 104.394) (end 175.1965 96.774) (width 0.25) (layer B.Cu) (net 1))
   (segment (start 142.1765 96.774) (end 142.1765 96.774) (width 0.25) (layer B.Cu) (net 1) (status 30))
-  (segment (start 142.1765 94.234) (end 144.7165 94.234) (width 0.25) (layer B.Cu) (net 2) (status 400000))
-  (segment (start 144.7165 94.234) (end 144.7165 91.694) (width 0.25) (layer B.Cu) (net 2) (status 800000))
+  (segment (start 142.1765 94.234) (end 144.7165 94.234) (width 0.25) (layer B.Cu) (net 2))
+  (segment (start 144.7165 94.234) (end 144.7165 91.694) (width 0.25) (layer B.Cu) (net 2))
   (segment (start 170.1165 86.614) (end 170.1165 89.154) (width 0.25) (layer B.Cu) (net 2))
   (segment (start 149.7965 91.694) (end 144.7165 91.694) (width 0.25) (layer B.Cu) (net 2))
@@
   (segment (start 190.4365 91.694) (end 192.9765 91.694) (width 0.25) (layer B.Cu) (net 4) (status 10))
   (segment (start 192.9765 89.154) (end 192.9765 91.694) (width 0.25) (layer B.Cu) (net 4))
-  (segment (start 192.9765 89.154) (end 198.0565 89.154) (width 0.25) (layer B.Cu) (net 4) (status 20))
+  (segment (start 192.9765 89.154) (end 195.5165 89.154) (width 0.25) (layer B.Cu) (net 4) (status 20))
   (segment (start 165.0365 86.614) (end 165.0365 96.774) (width 0.25) (layer B.Cu) (net 7))
   (segment (start 165.0365 96.774) (end 167.5765 96.774) (width 0.25) (layer B.Cu) (net 7))
-  (segment (start 187.8965 96.774) (end 187.8965 104.394) (width 0.25) (layer B.Cu) (net 16) (status 400000))
-  (segment (start 139.6365 110.744) (end 139.6365 106.934) (width 0.25) (layer B.Cu) (net 16) (status 800000))
+  (segment (start 187.8965 96.774) (end 187.8965 104.394) (width 0.25) (layer B.Cu) (net 16))
+  (segment (start 139.6365 110.744) (end 139.6365 106.934) (width 0.25) (layer B.Cu) (net 16))
   (via (at 139.6365 110.744) (size 0.6) (drill 0.4) (layers F.Cu B.Cu) (net 16))
   (segment (start 139.6365 127.254) (end 139.6365 110.744) (width 0.25) (layer F.Cu) (net 16))
@@
   (via (at 167.5765 114.554) (size 0.6) (drill 0.4) (layers F.Cu B.Cu) (net 23))
   (segment (start 167.5765 114.554) (end 167.5765 134.874) (width 0.25) (layer B.Cu) (net 23))
-  (segment (start 198.0565 96.774) (end 192.9765 96.774) (width 0.25) (layer B.Cu) (net 23) (status 10))
+  (segment (start 195.5165 96.774) (end 192.9765 96.774) (width 0.25) (layer B.Cu) (net 23) (status 10))
   (segment (start 192.9765 96.774) (end 192.9765 106.934) (width 0.25) (layer B.Cu) (net 23))
-  (segment (start 182.8165 109.474) (end 182.8165 112.014) (width 0.25) (layer B.Cu) (net 28) (status 400000))
+  (segment (start 182.8165 109.474) (end 182.8165 112.014) (width 0.25) (layer B.Cu) (net 28))
   (segment (start 152.3365 112.014) (end 152.3365 134.874) (width 0.25) (layer B.Cu) (net 28))
   (segment (start 182.8165 112.014) (end 152.3365 112.014) (width 0.25) (layer B.Cu) (net 28) (status 10))
